Commit message: Revert "abb irb 120 urdf"
This reverts commit 90a693af536e846c001faecab4fc68a623675f00.

File: ros_ws/st4_ws/src/abb_models/abb_irb120_support/urdf/iaac.urdf (robot description, URDF)
Before this commit: robot abb_irb120_3_58, 14 links, 14 joints
Links:
- removed link camera_body_link
- removed link camera_link
- link base_link: mass None -> 6.215; geometry collision mesh filename=package://abb_irb120_support/meshes/irb120_3_58/collision/b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; visual mesh filename=package://abb_irb120_support/meshes/irb120_3_58/visual/base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
Joints:
- removed joint cam_to_base_link
- removed joint cam_to_camlink
- removed joint tool0_to_cam
- joint tcp_joint: origin xyz=0.05 0 0.30 rpy=0 0 0 -> xyz=0 0 0.116 rpy=0 0 0

File: ros_ws/st4_ws/src/abb_models/abb_irb120_support/urdf/irb120_3_58.xacro (robot description, xacro)
@@ -2,6 +2,6 @@
 <robot name="abb_irb120_3_58" xmlns:xacro="http://ros.org/wiki/xacro">
   <xacro:include filename="$(find abb_irb120_support)/urdf/irb120_3_58_camera_ee_macro.xacro"/>
-  <xacro:include filename="$(find astra_camera)/urdf/astra_camera_macro.xacro">
+  <xacro:include filename="$(find astra_camera)/urdf/astra_camera_macro.xacro"/>
   <xacro:abb_irb120_3_58 prefix=""/>
-  <xacro:astra_camera prefix="">
+  <xacro:astra_camera prefix=""/>
 </robot>

File: ros_ws/st4_ws/src/abb_models/abb_irb120_support/urdf/irb120_3_58_macro.xacro (robot description, xacro)
@@ -278,4 +278,4 @@
     <link name="${prefix}tcp"/>
   </xacro:macro>
-<!--xacro:include filename="$(find astra_camera)/urdf/common_materials.xacro"/-->
+<xacro:include filename="$(find astra_camera)/urdf/common_materials.xacro"/>
 </robot>

File: ros_ws/st4_ws/src/abb_models/abb_irb120_support/urdf/test.urdf (robot description, URDF)
Before this commit: robot abb_irb120_3_58, 14 links, 14 joints
Links:
- removed link camera_link
- added link base_camera_link
- link base_link: mass None -> 6.215; geometry collision mesh filename=package://abb_irb120_support/meshes/irb120_3_58/collision/b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; visual mesh filename=package://abb_irb120_support/meshes/irb120_3_58/visual/base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
Joints:
- removed joint cam_to_base_link
- joint cam_to_camlink: child camera_link -> base_camera_link; origin xyz=0 0 0.025 rpy=0 -1.570795 0 -> xyz=0 0 0 rpy=0 0 0

File: ros_ws/st4_ws/src/ros_astra_camera/urdf/astra_camera_macro.xacro (robot description, xacro)
@@ -24,9 +24,9 @@
           </collision>
     </link>
-<joint type="fixed" name="${prefix}cam_body_to_table_link">
-        <origin xyz="-0.8 0 0" rpy="0 ${-pi*0.5} 0"/>
-        <parent link="${prefix}table_link"/>
-        <child link="${prefix}camera_body_link"/>
-        </joint>
+<joint type="fixed" name="${prefix}tool0_to_cam">
+    <origin xyz="0 0 0" rpy="0 0 0"/>
+    <parent link="${prefix}tool0"/>
+    <child link="${prefix}camera_body_link"/>
+    </joint>
 <joint type="fixed" name="${prefix}cam_to_camlink">
     <origin xyz="0 0 0.025" rpy="0 ${-pi*0.5} 0"/>
@@ -34,4 +34,10 @@
     <child link="${prefix}camera_link"/>
     </joint>
+<joint type="fixed" name="${prefix}cam_to_base_link">
+        <origin xyz="-0.8 0 0" rpy="0 ${-pi*0.5} 0"/>
+        <parent link="${prefix}camera_link"/>
+        <child link="${prefix}base_link"/>
+        </joint>
+<link name="${prefix}base_link"/>
 <link name="${prefix}camera_link"/>
  </xacro:macro>
