Commit message: urdf

File: ros_ws/st4_ws/src/abb_models/abb_irb120_support/urdf/static_wire_blade_ee.xacro (robot description, xacro)
@@ -26,5 +26,5 @@
   </link>
 <!-- DUMMY LINKS -->
-    <link name="${prefix}tcp"/>
+    <link name="${prefix}wire"/>
 <!-- DEFINE ADDED JOINTS -->
 <joint name="${prefix}link_6-tool" type="fixed">
@@ -37,5 +37,5 @@
    <origin xyz="0.05 0 0.30" rpy="0 0 0"/>
    <parent link="${prefix}tool0"/>
-   <child link="${prefix}tcp"/>
+   <child link="${prefix}wire"/>
  </joint>
     </xacro:macro>
