Commit message: abb irb 120 urdf
added and sorted camera and static tool links (TODO - positions)

File: ros_ws/st4_ws/src/abb_models/abb_irb120_support/urdf/irb120_3_58_basic.xacro (robot description, xacro)
@@ -4,4 +4,8 @@
   <xacro:macro name="abb_irb120_3_58" params="prefix">
     <!-- link list -->
+    <!-- DUMMY LINKS -->
+    <link name="${prefix}base"/>
+    <link name="${prefix}flange"/>
+     <!-- REAL LINKS -->
    <link name="${prefix}table_link">
   <inertial>
@@ -172,26 +176,5 @@
       </collision>
     </link>
-        <link name="${prefix}tool0">
-      <inertial>
-        <mass value="0.137"/>
-        <origin xyz="0 0 6.22E-05" rpy="0 0 6.22E-05"/>
-        <inertia ixx="0.001" ixy="0" ixz="0" iyy="0.001" iyz="0" izz="0.001"/>
-      </inertial>
-      <visual>
-        <origin xyz="0 0 6.22E-05" rpy="0 0 0"/>
-        <geometry>
-          <mesh filename="package://abb_irb120_support/meshes/irb120_3_58/visual/wire_cutter.stl"/>
-        </geometry>
-        <xacro:material_abb_black />
-      </visual>
-      <collision>
-        <origin xyz="0 0 6.22E-05" rpy="0 0 0"/>
-        <geometry>
-          <mesh filename="package://abb_irb120_support/meshes/irb120_3_58/collision/tool1_demo_collision.stl"/>
-        </geometry>
-        <xacro:material_abb_yellow />
-      </collision>
-    </link>
-    <!-- end of link list -->
+  <!-- end of link list -->
     <!-- joint list -->
     <joint name="${prefix}joint_1" type="revolute">
@@ -246,5 +229,4 @@
     <!--virtual links-->
     <!-- ROS-Industrial 'base' frame: base_link to ABB World Coordinates transform -->
-      <link name="${prefix}base"/>
     <joint name="${prefix}base-table" type="fixed">
       <origin xyz="0 0 0" rpy="0 0 0"/>
@@ -259,5 +241,4 @@
     </joint>
     <!-- ROS-Industrial 'flange' frame: attachment point for EEF models -->
-    <link name="${prefix}flange"/>
     <joint type="fixed" name="${prefix}joint_6-flange">
       <origin xyz="0 0 0" rpy="0 0 0"/>
@@ -265,17 +246,4 @@
       <child link="${prefix}flange"/>
     </joint>
-    <!-- ROS-Industrial 'tool0' frame: all-zeros tool frame -->
-    <joint name="${prefix}link_6-tool" type="fixed">
-      <origin xyz="0.001 0 0" rpy="0 ${radians (90)} 0" />
-      <parent link="${prefix}flange" />
-      <child link="${prefix}tool0" />
-    </joint>
-   <joint name="${prefix}tcp_joint" type="fixed">
-      <origin xyz="0.05 0 0.30" rpy="0 0 0"/>
-      <parent link="${prefix}tool0"/>
-      <child link="${prefix}tcp"/>
-    </joint>
-    <link name="${prefix}tcp"/>
-  </xacro:macro>
-<!--xacro:include filename="$(find astra_camera)/urdf/common_materials.xacro"/-->
+ </xacro:macro>
 </robot>

File: ros_ws/st4_ws/src/abb_models/abb_irb120_support/urdf/irb120_3_58_load_camera_and_robot.xacro (robot description, xacro)
@@ -2,6 +2,6 @@
 <robot name="abb_irb120_3_58" xmlns:xacro="http://ros.org/wiki/xacro">
   <xacro:include filename="$(find abb_irb120_support)/urdf/irb120_3_58_camera_ee_macro.xacro"/>
-  <xacro:include filename="$(find astra_camera)/urdf/astra_camera_macro.xacro"/>
+  <xacro:include filename="$(find astra_camera)/urdf/astra_camera_macro.xacro">
   <xacro:abb_irb120_3_58 prefix=""/>
-  <xacro:astra_camera prefix=""/>
+  <xacro:astra_camera prefix="">
 </robot>

File: ros_ws/st4_ws/src/abb_models/abb_irb120_support/urdf/tmp.urdf (robot description, URDF)
Before this commit: robot abb_irb120_3_58, 14 links, 14 joints
Links:
- link base_link: mass None -> 6.215; geometry collision mesh filename=package://abb_irb120_support/meshes/irb120_3_58/collision/b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; visual mesh filename=package://abb_irb120_support/meshes/irb120_3_58/visual/base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
Joints:
- removed joint cam_to_base_link
- removed joint tool0_to_cam
- added joint cam_body_to_table_link: type fixed, parent table_link, child camera_body_link, origin xyz=-0.8 0 0 rpy=0 -1.570795 0
- joint link_6-tool: parent flange -> table_link

File: ros_ws/st4_ws/src/ros_astra_camera/urdf/astra_camera_macro.xacro (robot description, xacro)
@@ -24,9 +24,9 @@
           </collision>
     </link>
-<joint type="fixed" name="${prefix}tool0_to_cam">
-    <origin xyz="0 0 0" rpy="0 0 0"/>
-    <parent link="${prefix}tool0"/>
-    <child link="${prefix}camera_body_link"/>
-    </joint>
+<joint type="fixed" name="${prefix}cam_body_to_table_link">
+        <origin xyz="-0.8 0 0" rpy="0 ${-pi*0.5} 0"/>
+        <parent link="${prefix}table_link"/>
+        <child link="${prefix}camera_body_link"/>
+        </joint>
 <joint type="fixed" name="${prefix}cam_to_camlink">
     <origin xyz="0 0 0.025" rpy="0 ${-pi*0.5} 0"/>
@@ -34,10 +34,4 @@
     <child link="${prefix}camera_link"/>
     </joint>
-<joint type="fixed" name="${prefix}cam_to_base_link">
-        <origin xyz="-0.8 0 0" rpy="0 ${-pi*0.5} 0"/>
-        <parent link="${prefix}camera_link"/>
-        <child link="${prefix}base_link"/>
-        </joint>
-<link name="${prefix}base_link"/>
 <link name="${prefix}camera_link"/>
  </xacro:macro>

Commit message: fix xacro

File: ros_ws/st4_ws/src/abb_models/abb_irb120_support/urdf/irb120_3_58_basic.xacro (robot description, xacro)
@@ -2,13 +2,38 @@
 <robot xmlns:xacro="http://ros.org/wiki/xacro">
   <xacro:include filename="$(find abb_resources)/urdf/common_materials.xacro"/>
-  <xacro:macro name="abb_irb120t_3_58" params="prefix">
+  <xacro:macro name="abb_irb120_3_58" params="prefix">
     <!-- link list -->
+    <!-- DUMMY LINKS -->
+    <link name="${prefix}base"/>
+    <link name="${prefix}flange"/>
+     <!-- REAL LINKS -->
+   <link name="${prefix}table_link">
+  <inertial>
+        <mass value="6.215"/>
+        <origin xyz="-0.04204 8.01E-05 0.07964" rpy="0 0 0"/>
+        <inertia ixx="0.0" ixy="0.0" ixz="0.0" iyy="0.0" iyz="0.0" izz="0.0"/>
+      </inertial>
+	<visual>
+        <origin xyz="0 0 0" rpy="0 0 0"/>
+        <geometry>
+          <mesh filename="package://abb_irb120_support/meshes/irb120_3_58/visual/table_iaac.stl"/>
+        </geometry>
+        <xacro:material_abb_orange />
+      </visual>
+      <collision>
+        <origin xyz="0 0 0" rpy="0 0 0"/>
+        <geometry>
+          <mesh filename="package://abb_irb120_support/meshes/irb120_3_58/collision/table_iaac.stl"/>
+        </geometry>
+        <xacro:material_abb_yellow />
+      </collision>
+    </link>
     <link name="${prefix}base_link">
-    	<inertial>
-    	  <mass value="6.215"/>
-    	  <origin xyz="-0.04204 8.01E-05 0.07964" rpy="0 0 0"/>
-    	  <inertia ixx="0.0247272" ixy="-8.0784E-05" ixz="0.00130902" iyy="0.0491285" iyz="-8.0419E-06" izz="0.0472376"/>
-    	</inertial>
-      <visual>
+  <inertial>
+        <mass value="6.215"/>
+        <origin xyz="-0.04204 8.01E-05 0.07964" rpy="0 0 0"/>
+        <inertia ixx="0.0" ixy="0.0" ixz="0.0" iyy="0.0" iyz="0.0" izz="0.0"/>
+      </inertial>
+	<visual>
         <origin xyz="0 0 0" rpy="0 0 0"/>
         <geometry>
@@ -26,9 +51,9 @@
     </link>
     <link name="${prefix}link_1">
-    	<inertial>
-    	  <mass value="3.067" />
-    	  <origin xyz="9.77E-05 -0.00012 0.23841" rpy="0 0 0"/>
-    	  <inertia ixx="0.0142175" ixy="-1.28579E-05" ixz="-2.31364E-05" iyy="0.0144041" iyz="1.93404E-05" izz="0.0104533"/>
-    	</inertial>
+      <inertial>
+        <mass value="3.067" />
+        <origin xyz="9.77E-05 -0.00012 0.23841" rpy="0 0 0"/>
+        <inertia ixx="0.0142175" ixy="-1.28579E-05" ixz="-2.31364E-05" iyy="0.0144041" iyz="1.93404E-05" izz="0.0104533"/>
+      </inertial>
       <visual>
         <origin xyz="0 0 0" rpy="0 0 0"/>
@@ -47,9 +72,9 @@
     </link>
     <link name="${prefix}link_2">
-    	<inertial>
-    	  <mass value="3.909"/>
-    	  <origin xyz="0.00078 -0.00212 0.10124" rpy="0 0 0"/>
-    	  <inertia ixx="0.0603111" ixy="9.83431E-06" ixz="5.72407E-05" iyy="0.041569" iyz="-0.00050497" izz="0.0259548"/>
-    	</inertial>
+      <inertial>
+        <mass value="3.909"/>
+        <origin xyz="0.00078 -0.00212 0.10124" rpy="0 0 0"/>
+        <inertia ixx="0.0603111" ixy="9.83431E-06" ixz="5.72407E-05" iyy="0.041569" iyz="-0.00050497" izz="0.0259548"/>
+      </inertial>
       <visual>
         <origin xyz="0 0 0" rpy="0 0 0"/>
@@ -68,9 +93,9 @@
     </link>
     <link name="${prefix}link_3">
-    	<inertial>
-    	  <mass value="2.944"/>
-    	  <origin xyz="0.02281 0.00106 0.05791" rpy="0 0 0"/>
-    	  <inertia ixx="0.00835606" ixy="-8.01545E-05" ixz="0.00142884" iyy="0.016713" iyz="-0.000182227" izz="0.0126984"/>
-    	</inertial>
+      <inertial>
+        <mass value="2.944"/>
+        <origin xyz="0.02281 0.00106 0.05791" rpy="0 0 0"/>
+        <inertia ixx="0.00835606" ixy="-8.01545E-05" ixz="0.00142884" iyy="0.016713" iyz="-0.000182227" izz="0.0126984"/>
+      </inertial>
       <visual>
         <origin xyz="0 0 0" rpy="0 0 0"/>
@@ -89,9 +114,9 @@
     </link>
     <link name="${prefix}link_4">
-    	<inertial>
-    	  <mass value="1.328"/>
-    	  <origin xyz="0.2247 0.00015 0.00041" rpy="0 0 0"/>
-    	  <inertia ixx="0.00284661" ixy="-2.12765E-05" ixz="-1.6435E-05" iyy="0.00401346" iyz="1.31336E-05" izz="0.0052535"/>
-    	</inertial>
+      <inertial>
+        <mass value="1.328"/>
+        <origin xyz="0.2247 0.00015 0.00041" rpy="0 0 0"/>
+        <inertia ixx="0.00284661" ixy="-2.12765E-05" ixz="-1.6435E-05" iyy="0.00401346" iyz="1.31336E-05" izz="0.0052535"/>
+      </inertial>
       <visual>
         <origin xyz="0 0 0" rpy="0 0 0"/>
@@ -110,9 +135,9 @@
     </link>
     <link name="${prefix}link_5">
-    	<inertial>
-    	  <mass value="0.546"/>
-    	  <origin xyz="-0.00109 3.68E-05 6.22E-05" rpy="0 0 0"/>
-    	  <inertia ixx="0.000404891" ixy="1.61943E-06" ixz="8.46805E-07" iyy="0.000892825" iyz="-1.51792E-08" izz="0.000815468"/>
-    	</inertial>
+      <inertial>
+        <mass value="0.546"/>
+        <origin xyz="-0.00109 3.68E-05 6.22E-05" rpy="0 0 0"/>
+        <inertia ixx="0.000404891" ixy="1.61943E-06" ixz="8.46805E-07" iyy="0.000892825" iyz="-1.51792E-08" izz="0.000815468"/>
+      </inertial>
       <visual>
         <origin xyz="0 0 0" rpy="0 0 0"/>
@@ -131,9 +156,9 @@
     </link>
     <link name="${prefix}link_6">
-    	<inertial>
-    	  <mass value="0.137"/>
-    	  <origin xyz="-0.00706 -0.00017 -1.32E-06" rpy="0 0 0"/>
-    	  <inertia ixx="0.001" ixy="0" ixz="0" iyy="0.001" iyz="0" izz="0.001"/>
-    	</inertial>
+      <inertial>
+        <mass value="0.137"/>
+        <origin xyz="-0.00706 -0.00017 -1.32E-06" rpy="0 0 0"/>
+        <inertia ixx="0.001" ixy="0" ixz="0" iyy="0.001" iyz="0" izz="0.001"/>
+      </inertial>
       <visual>
         <origin xyz="0 0 0" rpy="0 0 0"/>
@@ -151,5 +176,5 @@
       </collision>
     </link>
-    <!-- end of link list -->
+  <!-- end of link list -->
     <!-- joint list -->
     <joint name="${prefix}joint_1" type="revolute">
@@ -159,5 +184,5 @@
       <limit effort="0" lower="-2.87979" upper="2.87979" velocity="4.36332"/>
       <axis xyz="0 0 1"/>
-    	<dynamics damping="0.0" friction="0.0"/>
+      <dynamics damping="0.0" friction="0.0"/>
     </joint>
     <joint name="${prefix}joint_2" type="revolute">
@@ -167,5 +192,5 @@
       <limit effort="0" lower="-1.91986" upper="1.91986" velocity="4.36332"/>
       <axis xyz="0 1 0"/>
-    	<dynamics damping="0.0" friction="0.0"/>
+      <dynamics damping="0.0" friction="0.0"/>
     </joint>
     <joint name="${prefix}joint_3" type="revolute">
@@ -175,5 +200,5 @@
       <limit effort="0" lower="-1.91986" upper="1.22173" velocity="4.36332"/>
       <axis xyz="0 1 0"/>
-    	<dynamics damping="0.0" friction="0.0"/>
+      <dynamics damping="0.0" friction="0.0"/>
     </joint>
     <joint name="${prefix}joint_4" type="revolute">
@@ -181,7 +206,7 @@
       <parent link="${prefix}link_3"/>
       <child link="${prefix}link_4"/>
-      <limit effort="0" lower="-2.79253" upper="2.79253" velocity="7.33038"/>
+      <limit effort="0" lower="-2.79253" upper="2.79253" velocity="5.58505"/>
       <axis xyz="1 0 0"/>
-    	<dynamics damping="0.0" friction="0.0"/>
+      <dynamics damping="0.0" friction="0.0"/>
     </joint>
     <joint name="${prefix}joint_5" type="revolute">
@@ -189,7 +214,7 @@
       <parent link="${prefix}link_4"/>
       <child link="${prefix}link_5"/>
-      <limit effort="0" lower="-2.094395" upper="2.094395" velocity="10.29744"/>
+      <limit effort="0" lower="-2.094395" upper="2.094395" velocity="5.58505"/>
       <axis xyz="0 1 0"/>
-    	<dynamics damping="0.0" friction="0.0"/>
+      <dynamics damping="0.0" friction="0.0"/>
     </joint>
     <joint name="${prefix}joint_6" type="revolute">
@@ -197,18 +222,23 @@
       <parent link="${prefix}link_5"/>
       <child link="${prefix}link_6"/>
-      <limit effort="0" lower="-6.98132" upper="6.98132" velocity="10.471975"/>
+      <limit effort="0" lower="-6.98132" upper="6.98132" velocity="7.33038"/>
       <axis xyz="1 0 0"/>
-    	<dynamics damping="0.0" friction="0.0"/>
+      <dynamics damping="0.0" friction="0.0"/>
     </joint>
     <!-- end of joint list -->
+    <!--virtual links-->
     <!-- ROS-Industrial 'base' frame: base_link to ABB World Coordinates transform -->
-    <link name="${prefix}base" />
-    <joint name="${prefix}base_link-base" type="fixed">
+    <joint name="${prefix}base-table" type="fixed">
       <origin xyz="0 0 0" rpy="0 0 0"/>
-      <parent link="${prefix}base_link"/>
-      <child link="${prefix}base"/>
+      <parent link="${prefix}base"/>
+      <child link="${prefix}table_link"/>
+    </joint>
+      <!--link name="${prefix}base_link-table"/-->
+    <joint name="${prefix}base_link" type="fixed">
+      <origin xyz="0 0 0" rpy="0 0 0"/>
+      <parent link="${prefix}table_link"/>
+      <child link="${prefix}base_link"/>
     </joint>
     <!-- ROS-Industrial 'flange' frame: attachment point for EEF models -->
-    <link name="${prefix}flange"/>
     <joint type="fixed" name="${prefix}joint_6-flange">
       <origin xyz="0 0 0" rpy="0 0 0"/>
@@ -216,11 +246,4 @@
       <child link="${prefix}flange"/>
     </joint>
-    <!-- ROS-Industrial 'tool0' frame: all-zeros tool frame -->
-    <link name="${prefix}tool0" />
-    <joint name="${prefix}link_6-tool0" type="fixed">
-      <origin xyz="0 0 0" rpy="0 ${radians(90)} 0" />
-      <parent link="${prefix}flange" />
-      <child link="${prefix}tool0" />
-    </joint>
-  </xacro:macro>
+ </xacro:macro>
 </robot>

File: ros_ws/st4_ws/src/abb_models/abb_irb120_support/urdf/irb120_3_58_macro.xacro (robot description, xacro)
@@ -278,4 +278,4 @@
     <link name="${prefix}tcp"/>
   </xacro:macro>
-<xacro:include filename="$(find astra_camera)/urdf/common_materials.xacro"/>
+<!--xacro:include filename="$(find astra_camera)/urdf/common_materials.xacro"/-->
 </robot>

File: ros_ws/st4_ws/src/ros_astra_camera/urdf/astra_camera_macro.xacro (robot description, xacro)
@@ -24,7 +24,7 @@
           </collision>
     </link>
-<joint type="fixed" name="${prefix}tool0_to_cam">
+<joint type="fixed" name="${prefix}table_to_cam">
     <origin xyz="0 0 0" rpy="0 0 0"/>
-    <parent link="${prefix}tool0"/>
+    <parent link="${prefix}table_link"/>
     <child link="${prefix}camera_body_link"/>
     </joint>
@@ -34,10 +34,4 @@
     <child link="${prefix}camera_link"/>
     </joint>
-<joint type="fixed" name="${prefix}cam_to_base_link">
-        <origin xyz="-0.8 0 0" rpy="0 ${-pi*0.5} 0"/>
-        <parent link="${prefix}camera_link"/>
-        <child link="${prefix}base_link"/>
-        </joint>
-<link name="${prefix}base_link"/>
 <link name="${prefix}camera_link"/>
  </xacro:macro>

Commit message: camera calibration ver 1

File: ros_ws/st4_ws/src/abb_models/abb_irb120_support/urdf/irb120_3_58_basic.xacro (robot description, xacro)
@@ -178,4 +178,14 @@
   <!-- end of link list -->
     <!-- joint list -->
+    <joint name="${prefix}base_link" type="fixed">
+      <origin xyz="0 0 0" rpy="0 0 0"/>
+      <parent link="${prefix}table_link"/>
+      <child link="${prefix}base_link"/>
+    </joint>
+    <joint name="${prefix}base-table" type="fixed">
+      <origin xyz="0 0 0" rpy="0 0 0"/>
+      <parent link="${prefix}base"/>
+      <child link="${prefix}table_link"/>
+    </joint>
     <joint name="${prefix}joint_1" type="revolute">
       <origin rpy="0 0 0" xyz="0 0 0"/>
@@ -226,24 +236,14 @@
       <dynamics damping="0.0" friction="0.0"/>
     </joint>
+<joint type="fixed" name="${prefix}joint_6-flange">
+  <origin xyz="0 0 0" rpy="0 0 0"/>
+  <parent link="${prefix}link_6"/>
+  <child link="${prefix}flange"/>
+</joint>
     <!-- end of joint list -->
     <!--virtual links-->
     <!-- ROS-Industrial 'base' frame: base_link to ABB World Coordinates transform -->
-    <joint name="${prefix}base-table" type="fixed">
-      <origin xyz="0 0 0" rpy="0 0 0"/>
-      <parent link="${prefix}base"/>
-      <child link="${prefix}table_link"/>
-    </joint>
       <!--link name="${prefix}base_link-table"/-->
-    <joint name="${prefix}base_link" type="fixed">
-      <origin xyz="0 0 0" rpy="0 0 0"/>
-      <parent link="${prefix}table_link"/>
-      <child link="${prefix}base_link"/>
-    </joint>
     <!-- ROS-Industrial 'flange' frame: attachment point for EEF models -->
-    <joint type="fixed" name="${prefix}joint_6-flange">
-      <origin xyz="0 0 0" rpy="0 0 0"/>
-      <parent link="${prefix}link_6"/>
-      <child link="${prefix}flange"/>
-    </joint>
  </xacro:macro>
 </robot>

File: ros_ws/st4_ws/src/abb_models/abb_irb120_support/urdf/irb120_3_58_load_camera_and_robot.xacro (robot description, xacro)
@@ -2,6 +2,6 @@
 <robot name="abb_irb120_3_58" xmlns:xacro="http://ros.org/wiki/xacro">
   <xacro:include filename="$(find abb_irb120_support)/urdf/irb120_3_58_camera_ee_macro.xacro"/>
-  <xacro:include filename="$(find astra_camera)/urdf/astra_camera_macro.xacro">
+  <!--xacro:include filename="$(find astra_camera)/urdf/astra_camera_macro.xacro"-->
   <xacro:abb_irb120_3_58 prefix=""/>
-  <xacro:astra_camera prefix="">
+  <!--xacro:astra_camera prefix=""-->
 </robot>

File: ros_ws/st4_ws/src/abb_models/abb_irb120_support/urdf/irb120_3_58_load_robot_and_static_tool.xacro (robot description, xacro)
@@ -3,7 +3,7 @@
   <xacro:include filename="$(find abb_irb120_support)/urdf/irb120_3_58_basic.xacro"/>
   <xacro:include filename="$(find abb_irb120_support)/urdf/static_wire_blade_ee.xacro"/>
-  <xacro:include filename="$(find astra_camera)/urdf/astra_camera_macro.xacro"/>
+  <!--xacro:include filename="$(find astra_camera)/urdf/astra_camera_macro.xacro"/-->
   <xacro:abb_irb120_3_58 prefix=""/>
   <xacro:adding_static_tool prefix=""/>
-  <xacro:astra_camera prefix=""/>
+  <!--xacro:astra_camera prefix=""/-->
 </robot>

File: ros_ws/st4_ws/src/abb_models/abb_irb120_support/urdf/static_wire_blade_ee.xacro (robot description, xacro)
@@ -4,5 +4,5 @@
   <xacro:macro name="adding_static_tool" params="prefix">
 <!-- DEFINE ADDED LINKS -->
-      <link name="${prefix}tool0">
+      <link name="${prefix}tool_base">
     <inertial>
       <mass value="0.137"/>
@@ -30,11 +30,11 @@
 <joint name="${prefix}link_6-tool" type="fixed">
    <!--TODO: CHANGE SIZES AND LOCATION ACCORDING TO NEW TOOL-->
-    <origin xyz="0.001 0 0" rpy="0 ${radians (90)} 0" />
+    <origin xyz="0.3 -0.3 0" rpy="0 0 0" />
   <parent link="${prefix}table_link" />
-  <child link="${prefix}tool0" />
+  <child link="${prefix}tool_base" />
 </joint>
 <joint name="${prefix}tcp_joint" type="fixed">
-   <origin xyz="0.05 0 0.30" rpy="0 0 0"/>
-   <parent link="${prefix}tool0"/>
+   <origin xyz="0 0 0.5" rpy="0 0 0"/>
+   <parent link="${prefix}tool_base"/>
    <child link="${prefix}wire"/>
  </joint>

File: ros_ws/st4_ws/src/ros_astra_camera/urdf/astra_camera_macro.xacro (robot description, xacro)
@@ -4,5 +4,5 @@
  <xacro:macro name="astra_camera" params="prefix">
  <xacro:property name="pi" value="3.14159" />
-    <link name ="${prefix}camera_body_link">
+ <link name ="${prefix}camera_body_link">
      <inertial>
             <mass value="0.5"/>
@@ -24,15 +24,9 @@
           </collision>
     </link>
-<joint type="fixed" name="${prefix}table_to_cam">
-    <origin xyz="0 0 0" rpy="0 0 0"/>
-    <parent link="${prefix}table_link"/>
+<!--joint type="fixed" name="${prefix}cam_to_camlink">
+    <origin xyz="0 0 0.025" rpy="0 ${-pi*0.5} 0"/>
+    <parent link="${prefix}camera_link"/>
     <child link="${prefix}camera_body_link"/>
-    </joint>
-<joint type="fixed" name="${prefix}cam_to_camlink">
-    <origin xyz="0 0 0.025" rpy="0 ${-pi*0.5} 0"/>
-    <parent link="${prefix}camera_body_link"/>
-    <child link="${prefix}camera_link"/>
-    </joint>
-<link name="${prefix}camera_link"/>
+    </joint-->
  </xacro:macro>
 </robot>
